File: pcb/ws2812b/ws2812b.kicad_pcb (KiCad board)
At the start: 2 copper layers, 48.3 x 48.3 mm, 28 parts, among them J1 Jack-DC, J2 Jack-DC, J3 Conn_02x02_Top_Bottom, J4 Conn_01x04, J5 Conn_02x05_Top_Bottom, J6 Conn_01x02, U1 AMS1117-3.3, U2 ESP-12F, U3 STM32F103C8Tx, U4 74HC245

Commit message: Generate gerber files.
Routing:
- net 0: vias 14 -> 17
- added copper zone on B.Cu, net 0
- added copper zone on F.Cu, net 0
Other:
- board text added: "+3.3V"
- board text added: "BOOT0"
- board text added: "DATA"
- board text added: "GND"
- board text added: "GPIO0"
- board text added: "GPIO14"
- board text added: "GPIO16"
- board text added: "GPIO2"
- board text added: "NRST"
- board text added: "OUT"
- board text added: "RXD"
- board text added: "SWCLK"
- board text added: "SWDIO"
- board text added: "TXD"
- board text added: "USART1_RX"
- board text added: "USART1_TX"
- board text added: "ws2812b_v0.1 20190425"
Changed lines of the file:
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@@
-(kicad_pcb (version 20171130) (host pcbnew "(5.1.0)-1")
+(kicad_pcb (version 20171130) (host pcbnew "(5.1.0-0)")
   (general
     (thickness 1.6)
-    (drawings 6)
-    (tracks 358)
+    (drawings 25)
+    (tracks 362)
     (zones 0)
     (modules 28)
@@
     (0 F.Cu signal)
     (31 B.Cu signal)
-    (32 B.Adhes user)
-    (33 F.Adhes user)
+    (32 B.Adhes user hide)
+    (33 F.Adhes user hide)
     (34 B.Paste user)
     (35 F.Paste user)
@@
     (45 Margin user hide)
     (46 B.CrtYd user hide)
-    (47 F.CrtYd user)
+    (47 F.CrtYd user hide)
     (48 B.Fab user hide)
-    (49 F.Fab user)
+    (49 F.Fab user hide)
   )
   (setup
-    (last_trace_width 0.254)
+    (last_trace_width 0.25)
     (user_trace_width 0.254)
     (user_trace_width 0.508)
@@
     (visible_elements FFFFFF7F)
     (pcbplotparams
-      (layerselection 0x010fc_ffffffff)
+      (layerselection 0x010f0_ffffffff)
       (usegerberextensions false)
       (usegerberattributes false)
@@
       (outputformat 1)
       (mirror false)
-      (drillshape 1)
+      (drillshape 0)
       (scaleselection 1)
-      (outputdirectory ""))
+      (outputdirectory "gerber/"))
   )
   (net 0 "")
@@
     (tags "capacitor handsolder")
     (attr smd)
-    (fp_text reference C3 (at 0.254 2.54 270) (layer F.SilkS)
+    (fp_text reference C3 (at 2.159 -2.286 90) (layer F.SilkS)
       (effects (font (size 1 1) (thickness 0.15)))
     )
@@
     (tags "capacitor handsolder")
     (attr smd)
-    (fp_text reference C6 (at 0 -2.54 270) (layer F.SilkS)
+    (fp_text reference C6 (at 0.254 2.54 90) (layer F.SilkS)
       (effects (font (size 1 1) (thickness 0.15)))
     )
@@
     )
   )
+  (gr_text GND (at 91.44 36.83) (layer F.SilkS)
+    (effects (font (size 0.5 0.5) (thickness 0.1)))
+  )
+  (gr_text SWDIO (at 91.44 33.02) (layer F.SilkS)
+    (effects (font (size 0.5 0.5) (thickness 0.1)))
+  )
+  (gr_text SWCLK (at 91.44 30.48) (layer F.SilkS)
+    (effects (font (size 0.5 0.5) (thickness 0.1)))
+  )
+  (gr_text +3.3V (at 91.44 27.94) (layer F.SilkS)
+    (effects (font (size 0.5 0.5) (thickness 0.1)))
+  )
+  (gr_text OUT (at 53.975 70.485) (layer F.SilkS)
+    (effects (font (size 0.5 0.5) (thickness 0.1)))
+  )
+  (gr_text GND (at 53.975 67.31) (layer F.SilkS)
+    (effects (font (size 0.5 0.5) (thickness 0.1)))
+  )
+  (gr_text GPIO16 (at 64.77 60.325) (layer F.SilkS)
+    (effects (font (size 0.5 0.5) (thickness 0.1)))
+  )
+  (gr_text GPIO14 (at 64.77 57.785) (layer F.SilkS)
+    (effects (font (size 0.5 0.5) (thickness 0.1)))
+  )
+  (gr_text NRST (at 73.66 60.325) (layer F.SilkS)
+    (effects (font (size 0.5 0.5) (thickness 0.1)))
+  )
+  (gr_text BOOT0 (at 73.66 57.785) (layer F.SilkS)
+    (effects (font (size 0.5 0.5) (thickness 0.1)))
+  )
+  (gr_text GND (at 91.44 57.15 90) (layer F.SilkS)
+    (effects (font (size 0.5 0.5) (thickness 0.1)))
+  )
+  (gr_text +3.3V (at 88.9 57.15 90) (layer F.SilkS)
+    (effects (font (size 0.5 0.5) (thickness 0.1)))
+  )
+  (gr_text RXD (at 81.28 57.785 90) (layer F.SilkS)
+    (effects (font (size 0.5 0.5) (thickness 0.1)))
+  )
+  (gr_text TXD (at 83.82 57.785 90) (layer F.SilkS)
+    (effects (font (size 0.5 0.5) (thickness 0.1)))
+  )
+  (gr_text GPIO2 (at 91.44 66.04 90) (layer F.SilkS)
+    (effects (font (size 0.5 0.5) (thickness 0.1)))
+  )
+  (gr_text GPIO0 (at 88.9 66.04 90) (layer F.SilkS)
+    (effects (font (size 0.5 0.5) (thickness 0.1)))
+  )
+  (gr_text DATA (at 86.36 66.04 90) (layer F.SilkS)
+    (effects (font (size 0.5 0.5) (thickness 0.1)))
+  )
+  (gr_text USART1_RX (at 83.82 66.675 90) (layer F.SilkS)
+    (effects (font (size 0.5 0.5) (thickness 0.1)))
+  )
+  (gr_text USART1_TX (at 81.28 66.675 90) (layer F.SilkS)
+    (effects (font (size 0.5 0.5) (thickness 0.1)))
+  )
+  (gr_text "ws2812b_v0.1\n20190425" (at 88.9 71.755) (layer F.SilkS)
+    (effects (font (size 0.5 0.5) (thickness 0.1)))
+  )
   (gr_line (start 66.5226 55.2958) (end 65.9892 54.737) (layer F.SilkS) (width 0.12))
-  (gr_circle (center 66.548 29.21) (end 66.548 30.988) (layer B.SilkS) (width 0.12))
   (gr_line (start 99.06 25.4) (end 50.8 25.4) (layer Edge.Cuts) (width 0.05))
   (gr_line (start 99.06 73.66) (end 99.06 25.4) (layer Edge.Cuts) (width 0.05))
   (gr_line (start 50.8 73.66) (end 99.06 73.66) (layer Edge.Cuts) (width 0.05))
   (gr_line (start 50.8 25.4) (end 50.8 73.66) (layer Edge.Cuts) (width 0.05))
-  (via (at 93.472 69.85) (size 5) (drill 3.5) (layers F.Cu B.Cu) (net 0))
+  (via (at 94.615 69.215) (size 5) (drill 3.5) (layers F.Cu B.Cu) (net 0))
   (segment (start 66.548 55.2704) (end 66.4972 55.2704) (width 0.254) (layer F.Cu) (net 0))
   (segment (start 87.45151 46.50099) (end 87.4745 46.478) (width 0.254) (layer B.Cu) (net 1))
@@
   (segment (start 68.79 66.813) (end 69.919 66.813) (width 0.254) (layer B.Cu) (net 2))
   (segment (start 70.612 67.506) (end 70.612 71.374) (width 0.254) (layer B.Cu) (net 2))
-  (segment (start 71.251 72.013) (end 75.99 72.013) (width 0.254) (layer B.Cu) (net 2))
+  (segment (start 71.251 72.013) (end 72.767 72.013) (width 0.254) (layer B.Cu) (net 2))
   (segment (start 70.612 71.374) (end 71.251 72.013) (width 0.254) (layer B.Cu) (net 2))
   (segment (start 65.748 34.535) (end 64.516 35.767) (width 0.508) (layer B.Cu) (net 2))
@@
   (segment (start 90.17 35.814) (end 91.44 34.544) (width 1.524) (layer B.Cu) (net 2))
   (via (at 90.17 35.814) (size 0.8) (drill 0.4) (layers F.Cu B.Cu) (net 2))
+  (via (at 78.74 71.755) (size 0.8) (drill 0.4) (layers F.Cu B.Cu) (net 2))
+  (segment (start 72.767 72.013) (end 75.99 72.013) (width 0.254) (layer B.Cu) (net 2))
+  (via (at 72.767 72.013) (size 0.8) (drill 0.4) (layers F.Cu B.Cu) (net 2))
+  (via (at 78.74 50.8) (size 0.8) (drill 0.4) (layers F.Cu B.Cu) (net 2))
   (segment (start 61.976 58.166) (end 60.96 57.15) (width 0.254) (layer B.Cu) (net 3))
   (segment (start 60.96 32.385) (end 60.96 32.512) (width 1.524) (layer B.Cu) (net 3))
@@
   (segment (start 68.79 67.463) (end 67.661 67.463) (width 0.254) (layer B.Cu) (net 11))
   (segment (start 67.661 67.463) (end 67.056 68.068) (width 0.254) (layer B.Cu) (net 11))
-  (segment (start 84.062 57.9) (end 86.36 60.198) (width 0.254) (layer B.Cu) (net 79))
-  (segment (start 84.062 50.3905) (end 84.062 57.9) (width 0.254) (layer B.Cu) (net 79))
-  (segment (start 77.119 66.813) (end 75.99 66.813) (width 0.254) (layer B.Cu) (net 78))
-  (segment (start 83.487081 66.813) (end 77.119 66.813) (width 0.254) (layer B.Cu) (net 78))
-  (segment (start 86.36 63.940081) (end 83.487081 66.813) (width 0.254) (layer B.Cu) (net 78))
-  (segment (start 86.36 62.738) (end 86.36 63.940081) (width 0.254) (layer B.Cu) (net 78))
   (segment (start 88.614 37.902) (end 87.864 37.902) (width 0.254) (layer F.Cu) (net 12))
   (segment (start 94.544 37.902) (end 87.864 37.902) (width 0.254) (layer F.Cu) (net 12))
@@
   (segment (start 91.313 49.902) (end 91.44 50.029) (width 0.254) (layer F.Cu) (net 20))
   (segment (start 87.864 49.902) (end 91.313 49.902) (width 0.254) (layer F.Cu) (net 20))
+  (segment (start 77.119 66.813) (end 75.99 66.813) (width 0.254) (layer B.Cu) (net 78))
+  (segment (start 83.487081 66.813) (end 77.119 66.813) (width 0.254) (layer B.Cu) (net 78))
+  (segment (start 86.36 63.940081) (end 83.487081 66.813) (width 0.254) (layer B.Cu) (net 78))
+  (segment (start 86.36 62.738) (end 86.36 63.940081) (width 0.254) (layer B.Cu) (net 78))
+  (segment (start 84.062 57.9) (end 86.36 60.198) (width 0.254) (layer B.Cu) (net 79))
+  (segment (start 84.062 50.3905) (end 84.062 57.9) (width 0.254) (layer B.Cu) (net 79))
   (zone (net 0) (net_name "") (layers F&B.Cu) (hatch edge 0.508)
     (connect_pads (clearance 0.508))
@@
       )
     )
+  )
+  (zone (net 2) (net_name 0) (layer F.Cu) (hatch edge 0.508)
+    (connect_pads (clearance 0.508))
+    (min_thickness 0.254)
+    (fill yes (arc_segments 32) (thermal_gap 0.508) (thermal_bridge_width 0.508))
+    (polygon
+      (pts
+        (xy 50.8 25.4) (xy 50.8 73.66) (xy 99.06 73.66) (xy 99.06 25.4)
+      )
+    )
+  )
+  (zone (net 2) (net_name 0) (layer B.Cu) (hatch edge 0.508)
+    (connect_pads (clearance 0.508))
+    (min_thickness 0.254)
+    (fill yes (arc_segments 32) (thermal_gap 0.508) (thermal_bridge_width 0.508))
+    (polygon
+      (pts
+        (xy 50.8 25.4) (xy 50.8 73.66) (xy 99.06 73.66) (xy 99.06 25.4)
+      )
+    )
